Commit message: Use Iron Man colors

File: urdf/my_robot.xacro (robot description, xacro)
@@ -173,17 +173,17 @@
   </joint>
   <gazebo reference="left_wheel">
-    <material>Gazebo/Green</material>
+    <material>Gazebo/Gold</material>
   </gazebo>
   <gazebo reference="right_wheel">
-    <material>Gazebo/Green</material>
+    <material>Gazebo/Gold</material>
   </gazebo>
   <gazebo reference="chassis">
-    <material>Gazebo/Blue</material>
+    <material>Gazebo/Red</material>
   </gazebo>
   <gazebo reference="camera">
-    <material>Gazebo/Red</material>
+    <material>Gazebo/BlueGlow</material>
   </gazebo>
-  <gazebo reference="left_wheel">
-    <material>Gazebo/Green</material>
+  <gazebo reference="hokuyo">
+    <material>Gazebo/Gold</material>
   </gazebo>
   <xacro:include filename="$(find my_robot)/urdf/my_robot.gazebo" />

Commit message: Upgrade to Kinect from RGB camera

File: urdf/my_robot.xacro (robot description, xacro)
@@ -172,4 +172,11 @@
     <axis xyz="0 1 0"/>
   </joint>
+  <joint name="camera_optical_joint" type="fixed">
+    <origin xyz="0 0 0" rpy="-1.5707 0 -1.5707"/>
+    <parent link="camera"/>
+    <child link="camera_link_optical"/>
+  </joint>
+  <link name="camera_link_optical">
+  </link>
   <gazebo reference="left_wheel">
     <material>Gazebo/Gold</material>

Commit message: Fix link and frame names

File: urdf/my_robot.xacro (robot description, xacro)
@@ -175,7 +175,7 @@
     <origin xyz="0 0 0" rpy="-1.5707 0 -1.5707"/>
     <parent link="camera"/>
-    <child link="camera_link_optical"/>
+    <child link="camera_link"/>
   </joint>
-  <link name="camera_link_optical">
+  <link name="camera_link">
   </link>
   <gazebo reference="left_wheel">

Commit message: Fix camera orientation

File: urdf/my_robot.xacro (robot description, xacro)
@@ -173,5 +173,5 @@
   </joint>
   <joint name="camera_optical_joint" type="fixed">
-    <origin xyz="0 0 0" rpy="-1.5707 0 -1.5707"/>
+    <origin xyz="0 0 0" rpy="0 0 0"/>
     <parent link="camera"/>
     <child link="camera_link"/>

Commit message: Fix camera references

File: urdf/my_robot.xacro (robot description, xacro)
@@ -1,4 +1,5 @@
 <?xml version='1.0'?>
 <robot name="my_robot" xmlns:xacro="http://www.ros.org/wiki/xacro">
+  <xacro:include filename="$(find my_robot)/urdf/my_robot.gazebo" />
   <link name="robot_footprint"></link>
   <joint name="robot_footprint_joint" type="fixed">
@@ -139,9 +140,17 @@
     </inertial>
   </link>
-  <joint type="fixed" name="camera_joint">
+  <joint name="camera_joint" type="fixed" >
+    <axis xyz="0 1 0"/>
     <origin xyz="0.2 0 0" rpy="0 0 0"/>
+    <parent link="chassis"/>
     <child link="camera"/>
-    <parent link="chassis"/>
   </joint>
+  <joint name="camera_optical_joint" type="fixed">
+    <origin xyz="0 0 0" rpy="-1.5707 0 -1.5707"/>
+    <parent link="camera"/>
+    <child link="camera_link_optical"/>
+  </joint>
+  <link name="camera_link_optical">
+  </link>
   <link name='hokuyo'>
     <collision>
@@ -172,11 +181,4 @@
     <axis xyz="0 1 0"/>
   </joint>
-  <joint name="camera_optical_joint" type="fixed">
-    <origin xyz="0 0 0" rpy="0 0 0"/>
-    <parent link="camera"/>
-    <child link="camera_link"/>
-  </joint>
-  <link name="camera_link">
-  </link>
   <gazebo reference="left_wheel">
     <material>Gazebo/Gold</material>
@@ -194,4 +196,3 @@
     <material>Gazebo/Gold</material>
   </gazebo>
-  <xacro:include filename="$(find my_robot)/urdf/my_robot.gazebo" />
 </robot>
